Commit message: added TF node and launch file

File: can_devices/sdv_control_ros2/models/el_rasho.urdf (robot description, URDF)
Before this commit: robot sdv, 1 links, 0 joints
Links:
- link sdv: geometry visual mesh filename=package://sdv_control_ros2/models/meshes/el_rasho.stl scale=0.03 0.03 0.03
