Commit message: tf2 broadcaster compiles and rviz model recently added

File: docker_ws/sdv_description/urdf/sdv.urdf (robot description, URDF)
Before this commit: robot sdv, 15 links, 14 joints
Links:
- removed link base_footprint
- removed link base_laser_front_link
- removed link caster_link_bl
- removed link caster_link_br
- removed link caster_link_fl
- removed link caster_link_fr
- removed link plate_link
- removed link virtual_link_xy
- removed link virtual_link_yz
- removed link wheel_link_bl
- removed link wheel_link_br
- removed link wheel_link_fl
- removed link wheel_link_fr
- removed link world
- link base_link: mass 22.0 -> None; geometry visual mesh filename=package://sdv_description/meshes/sdv.stl scale=1.0 1.0 1.0
Joints:
- removed joint base_footprint_joint
- removed joint base_laser_front_hokuyo_urg04_laser_joint
- removed joint caster_joint_bl
- removed joint caster_joint_br
- removed joint caster_joint_fl
- removed joint caster_joint_fr
- removed joint plate_joint
- removed joint virtual_joint_x
- removed joint virtual_joint_y
- removed joint virtual_joint_z
- removed joint wheel_joint_bl
- removed joint wheel_joint_br
- removed joint wheel_joint_fl
- removed joint wheel_joint_fr

Commit message: checking offsets. wrong results

File: docker_ws/sdv_description/urdf/sdv.urdf (robot description, URDF)
Before this commit: robot sdv, 1 links, 0 joints
Links:
- removed link base_link
- added link sdv_base_link; visual mesh filename=package://sdv_description/meshes/sdv.stl scale=1.0 1.0 1.0

Commit message: almost ready for real tests

File: docker_ws/sdv_description/urdf/sdv.urdf (robot description, URDF)
Before this commit: robot sdv, 1 links, 0 joints
Links:
- removed link sdv_base_link
- added link base_link; visual mesh filename=package://sdv_description/meshes/sdv.stl scale=1.0 1.0 1.0

Commit message: nav2 settings for final implementation

File: docker_ws/sdv_description/urdf/sdv.urdf (robot description, URDF)
Before this commit: robot sdv, 1 links, 0 joints
Links:
- link base_link: geometry collision mesh filename=package://sdv_description/meshes/sdv_nav.stl scale=1.0 1.0 1.0; visual mesh filename=package://sdv_description/meshes/sdv_nav.stl scale=1.0 1.0 1.0
