Commit message: Initial interpolation, falta limpiar

File: workspace/src/sdv_description/urdf/sdv.urdf (robot description, URDF)
Before this commit: robot sdv, 1 links, 0 joints
Links:
- added link front
Joints:
- added joint base_to_front: type fixed, parent base_link, child front, origin xyz=1.2 0 0
