Commit message: new docker with pytorch, made rviz great again

File: workspace/src/sdv_description/urdf/sdv_simple_NED.urdf (robot description, URDF)
Before this commit: robot sdv, 1 links, 0 joints
Links:
- removed link sdv
- added link base_link; visual mesh filename=package://sdv_description/meshes/sdv.stl scale=1.0 1.0 1.0
